Commit message: new name for analytic_throw and change urdf flexpicker gripper

File: code/urdf/flexpicker.urdf (robot description, URDF)
Before this commit: robot flexpicker, 10 links, 9 joints
Joints:
- joint l_gripper_l_finger_joint: limit lower=-0.04 upper=0.04 effort=25.0 velocity=2.0 -> lower=-0.04 upper=0.04 effort=25.0 velocity=10
- joint l_gripper_r_finger_joint: limit lower=-0.04 upper=0.04 effort=25.0 velocity=2.0 -> lower=-0.04 upper=0.04 effort=25.0 velocity=10
